Commit message: Update of urdfs for simulation

File: robotino_description/urdf/robotino.urdf.xacro (robot description, xacro)
@@ -1,6 +1,6 @@
 <?xml version="1.0"?>
 <robot name="robotino" xmlns:xacro="http://wiki.ros.org/xacro">
+  <xacro:include filename="$(find robotino_description)/urdf/robotino_parts.urdf.xacro"/>
   <xacro:include filename="$(find robotino_description)/urdf/robotino_body.urdf.xacro"/>
-  <xacro:include filename="$(find robotino_description)/urdf/robotino_parts.urdf.xacro"/>
-  <robotino_body/>
+  <xacro:robotino_body/>
 </robot>

File: robotino_description/urdf/robotino_body.urdf.xacro (robot description, xacro)
@@ -32,27 +32,26 @@
         </link>
         <gazebo reference="base_link">
-            <material>Gazebo/White</material>
             <turnGravityOff>false</turnGravityOff>
         </gazebo>
         <!-- wheels -->
-        <wheel name="wheel0" parent="base_link">
+        <xacro:wheel name="wheel0" parent="base_link">
             <origin xyz="0.065 0.11 0.04" rpy="0 0 ${M_PI/3}"/>
             <axis xyz="-1 0 0"/>
-        </wheel>
-        <wheel name="wheel1" parent="base_link">
+        </xacro:wheel >
+        <xacro:wheel  name="wheel1" parent="base_link">
             <origin xyz="-0.13 0 0.04" rpy="0 0 0"/>
             <axis xyz="1 0 0"/>
-        </wheel>
-        <wheel name="wheel2" parent="base_link">
+        </xacro:wheel >
+        <xacro:wheel  name="wheel2" parent="base_link">
             <origin xyz="0.065 -0.11 0.04" rpy="0 0 -${M_PI/3}"/>
             <axis xyz="-1 0 0"/>
-        </wheel>
+        </xacro:wheel >
         <!-- others -->
-        <command_bridge name="command_bridge" parent="base_link">
+        <xacro:command_bridge name="command_bridge" parent="base_link">
             <origin xyz="-0.05 0 0.13" rpy="0 0 ${M_PI/2}"/>
-        </command_bridge>
-        <anglebracketusb name="anglebracketusb" parent="base_link">
+        </xacro:command_bridge>
+        <!-- <xacro:anglebracketusb name="anglebracketusb" parent="base_link">
             <origin xyz="0.008 0 0.137" rpy="0 0 ${M_PI/2}"/>
-        </anglebracketusb>
+        </xacro:anglebracketusb> -->
         <!-- gazebo control -->
         <gazebo>
@@ -63,4 +62,5 @@
                 <odometryRate>20</odometryRate>
                 <robotBaseFrame>base_link</robotBaseFrame>
+                <publishTF>true</publishTF>
             </plugin>
             <plugin name="gazebo_ros_control" filename="libgazebo_ros_control.so"/>

File: robotino_description/urdf/robotino_parts.urdf.xacro (robot description, xacro)
@@ -5,4 +5,7 @@
     <xacro:property name="PLATFORM_HEIGHT" value="0.58"/>
     <xacro:property name="PLATFORM_RADIUS" value="0.22"/>
+    <material name="dark_grey">
+        <color rgba="${150/255} ${150/255} ${150/255} 1.0"/>
+    </material>
     <!-- wheel -->
     <xacro:macro name="wheel" params="parent name *origin *axis">
@@ -21,21 +24,24 @@
         </link>
         <gazebo reference="${name}_link">
-            <material>Gazebo/Yellow</material>
+            <material>Gazebo/Grey</material>
             <turnGravityOff>false</turnGravityOff>
         </gazebo>
-        <joint name="${name}_joint" type="continuous">
-            <insert_block name="origin" />
-            <insert_block name="axis"/>
+        <joint name="${name}_joint" type="fixed">
+            <xacro:insert_block name="origin" />
+            <xacro:insert_block name="axis"/>
             <parent link="${parent}"/>
             <child link="${name}_link"/>
         </joint>
-        <transmission name="${name}_joint_trans">
-            <type>transmissio_interface/SimpleTransmission</type>
-            <joint name="${name}_joint"/>
+        <!-- ToDo: Comment out and use to turn the mecanum -->
+        <!-- <transmission name="${name}_joint_trans">
+            <type>transmission_interface/SimpleTransmission</type>
+            <joint name="${name}_joint">
+                <hardwareInterface>EffortJointInterface</hardwareInterface>
+            </joint>
             <actuator name="${name}_motor">
                 <hardwareInterface>EffortJointInterface</hardwareInterface>
                 <mechanicalReducation>1</mechanicalReducation>
             </actuator>
-        </transmission>
+        </transmission> -->
     </xacro:macro>
     <!-- command bridge -->
@@ -55,5 +61,5 @@
         </link>
         <joint name="${name}_joint" type="fixed">
-            <insert_block name="origin"/>
+            <xacro:insert_block name="origin"/>
             <parent link="${parent}"/>
             <child link="${name}_link"/>
@@ -76,5 +82,5 @@
         </link>
         <joint name="${name}_joint" type="fixed">
-            <insert_block name="origin"/>
+            <xacro:insert_block name="origin"/>
             <parent link="${parent}"/>
             <child link="${name}_link"/>
@@ -104,5 +110,58 @@
         </link>
         <joint name="${name}_joint" type="fixed">
-            <insert_block name="origin"/>
+            <xacro:insert_block name="origin"/>
+            <parent link="${parent}"/>
+            <child link="${name}_link"/>
+        </joint>
+    </xacro:macro>
+    <!-- Lochplatte -->
+    <xacro:macro name="plate" params="parent name">
+        <link name="${name}_link">
+            <inertial>
+                <mass value="0.00001"/>
+                <origin xyz="0 0 0"/>
+                <inertia ixx="1.0" ixy="0.0" ixz="0.0" iyy="1.0" iyz="0.0" izz="1.0"/>
+            </inertial>
+            <visual>
+                <origin xyz="0 0 0.12"/>
+                <geometry>
+                    <box size="0.002 0.06 0.24"/>
+                </geometry>
+                <material name="dark_grey"/>
+            </visual>
+        </link>
+        <gazebo reference="${name}_link">
+            <material>Gazebo/Grey</material>
+            <turnGravityOff>false</turnGravityOff>
+        </gazebo>
+        <joint name="${name}_joint" type="fixed">
+            <!-- <xacro:insert_block name="origin"/> -->
+            <origin xyz="0.05 0 0.07"/>
+            <parent link="${parent}"/>
+            <child link="${name}_link"/>
+        </joint>
+    </xacro:macro>
+    <!-- Bracket -->
+    <xacro:macro name="bracket" params="parent name scale *origin">
+        <link name="${name}_link">
+            <inertial>
+                <mass value="0.00001"/>
+                <origin xyz="0 0 0"/>
+                <inertia ixx="1.0" ixy="0.0" ixz="0.0" iyy="1.0" iyz="0.0" izz="1.0"/>
+            </inertial>
+            <visual>
+                <origin xyz="0 0 0" rpy="0 0 0"/>
+                <geometry>
+                    <mesh filename="package://robotino_description/meshes/parts/bracket.dae" scale="0.001 ${scale} ${scale}"/>
+                </geometry>
+                <material name="dark_grey"/>
+            </visual>
+        </link>
+        <gazebo reference="${name}_link">
+            <material>Gazebo/DarkGrey</material>
+            <turnGravityOff>false</turnGravityOff>
+        </gazebo>
+        <joint name="${name}_joint" type="fixed">
+            <xacro:insert_block name="origin"/>
             <parent link="${parent}"/>
             <child link="${name}_link"/>

File: robotino_description/urdf/robotino_platform.urdf.xacro (robot description, xacro)
@@ -3,8 +3,8 @@
     <xacro:include filename="$(find robotino_description)/urdf/robotino_body.urdf.xacro"/>
     <xacro:include filename="$(find robotino_description)/urdf/robotino_parts.urdf.xacro"/>
-    <robotino_body/>
+    <xacro:robotino_body/>
     <!-- add platform -->
-    <platform name="platform" parent="base_link">
+    <xacro:platform name="platform" parent="base_link">
         <origin xyz="0.0 0.0 0.13" rpy="0 0 0"/>
-    </platform>
+    </xacro:platform>
 </robot>

File: robotino_description/urdf/sensors/asus_xtion_pro.urdf.xacro (robot description, xacro)
@@ -1,11 +1,11 @@
 <?xml version="1.0"?>
 <robot name="sensor_asus_xtion_pro" xmlns:xacro="http://ros.org/wiki/xacro">
-  <xacro:include filename="$(find robotino_description)/urdf/3dsensor_gazebo.urdf.xacro"/>
-  <xacro:property name="M_SCALE" value="0.001"/>
+  <xacro:include filename="$(find robotino_description)/urdf/sensors/3dsensor_gazebo.urdf.xacro"/>
+  <xacro:property name="M_SCALE2" value="0.001"/>
   <xacro:property name="asus_xtion_pro_depth_rel_rgb_py" value="0.0270" />
   <xacro:property name="asus_xtion_pro_cam_rel_rgb_py"   value="-0.0220" />
-  <xacro:property name="cam_px" value="0.0"/>
-  <xacro:property name="cam_py" value="0.0"/>
-  <xacro:property name="cam_pz" value="0.0"/>
+  <xacro:property name="cam_px" value="0.10"/>
+  <xacro:property name="cam_py" value="0.014"/>
+  <xacro:property name="cam_pz" value="0.283"/>
   <xacro:property name="cam_or" value="0.0"/>
   <xacro:property name="cam_op" value="0.0"/>
@@ -51,5 +51,5 @@
         <origin xyz="-0.01 0 0" rpy="${-M_PI/2} -${M_PI} ${-M_PI/2}"/>
         <geometry>
-          <mesh filename="package://robotino_description/meshes/sensors/asus_xtion_pro_live.dae" scale="${M_SCALE} ${M_SCALE} ${M_SCALE}"/>
+          <mesh filename="package://robotino_description/meshes/sensors/asus_xtion_pro_live.dae" scale="${M_SCALE2} ${M_SCALE2} ${M_SCALE2}"/>
         </geometry>
       </visual>
@@ -97,5 +97,5 @@
     </link>
     <!-- RGBD sensor for simulation, same as Kinect -->
-    <sim_3dsensor/>
+    <xacro:sim_3dsensor/>
   </xacro:macro>
 </robot>

File: robotino_description/urdf/sensors/hokuyo.urdf.xacro (robot description, xacro)
@@ -1,4 +1,4 @@
 <?xml version="1.0"?>
-<robot name="sensor_hokuyo" xmlns:xacro="http://wiki.ros.org/xacro">
+<root xmlns:xacro="http://www.ros.org/wiki/xacro">
   <xacro:property name="M_PI" value="3.14159"/>
   <xacro:property name="M_SCALE" value="0.01"/>
@@ -7,5 +7,5 @@
   <xacro:macro name="hokuyo" params="parent name *origin">
     <joint name="${name}_joint" type="fixed">
-      <insert_block name="origin" />
+      <xacro:insert_block name="origin" />
       <parent link="${parent}"/>
       <child link="${name}_link" />
@@ -16,12 +16,11 @@
         <origin xyz="0 0 0" />
         <inertia ixx="1.0" ixy="0.0" ixz="0.0"
-          iyy="1.0" iyz="0.0"
-          izz="1.0" />
+		 iyy="1.0" iyz="0.0"
+		 izz="1.0" />
       </inertial>
       <visual>
-        <origin xyz="0 0 0" rpy="0 0 ${M_PI/2}" />
+        <origin xyz="0 0 -0.05" rpy="0 0 ${M_PI/2}" />
         <geometry>
-          <mesh
-filename="package://robotino_description/meshes/sensors/hokuyo.dae" scale="${M_SCALE} ${M_SCALE} ${M_SCALE}"/>
+          <mesh filename="package://robotino_description/meshes/sensors/hokuyo.dae" scale="${M_SCALE} ${M_SCALE} ${M_SCALE}"/>
         </geometry>
       </visual>
@@ -33,4 +32,41 @@
       </collision>
     </link>
+    <!-- gazebo extensions -->
+    <xacro:hokuyo_gazebo name="${name}" ros_topic="scan" update_rate="10" min_angle="-1.570796" max_angle="1.570796"/>
   </xacro:macro>
-</robot>
+  <!--GAZEBO PLUGIN-->
+  <xacro:macro name="hokuyo_gazebo" params="name ros_topic update_rate min_angle max_angle">
+    <gazebo reference="${name}_link">
+      <sensor name="${name}" type="gpu_ray">
+        <!--always_on>true</always_on-->
+        <update_rate>40</update_rate>
+        <pose>0 0 0 0 0 0</pose>
+        <visualize>false</visualize>
+        <ray>
+          <scan>
+            <horizontal>
+              <samples>683</samples>
+              <resolution>0.36</resolution>
+              <min_angle>-2,0944</min_angle>
+              <max_angle>2,0944</max_angle>
+            </horizontal>
+          </scan>
+          <range>
+            <min>0.03</min>
+            <max>5.6</max>
+            <resolution>0.01</resolution>
+          </range>
+          <noise>
+            <type>gaussian</type>
+            <mean>0.0</mean>
+            <stddev>0.005</stddev>
+          </noise>
+        </ray>
+        <plugin name="gazebo_ros_${name}_controller" filename="libgazebo_ros_gpu_laser.so">
+          <topicName>${ros_topic}</topicName>
+          <frameName>${name}_link</frameName>
+        </plugin>
+      </sensor>
+    </gazebo>
+  </xacro:macro>
+</root>
