Commit message: Renamed all files containing robotino to rto

File: rto_description/urdf/rto-1.urdf (robot description, URDF)
Before this commit: robot robotino, 11 links, 10 joints
Links:
- link base_link: geometry collision cylinder length=0.05 radius=0.18; visual mesh filename=package://rto_description/meshes/parts/rto_base.dae scale=0.01 0.01 0.01
- link wheel0_link: geometry visual mesh filename=package://rto_description/meshes/parts/rto_wheel.dae scale=0.01 0.01 0.01
- link wheel1_link: geometry visual mesh filename=package://rto_description/meshes/parts/rto_wheel.dae scale=0.01 0.01 0.01
- link wheel2_link: geometry visual mesh filename=package://rto_description/meshes/parts/rto_wheel.dae scale=0.01 0.01 0.01

File: rto_description/urdf/rto-1.urdf.xacro (robot description, xacro)
@@ -1,9 +1,9 @@
 <?xml version="1.0"?>
-<robot name="robotino" xmlns:xacro="http://wiki.ros.org/xacro">
-  <xacro:include filename="$(find rto_description)/urdf/robotino_parts.urdf.xacro"/>
-  <xacro:include filename="$(find rto_description)/urdf/robotino_body.urdf.xacro"/>
+<robot name="rto" xmlns:xacro="http://wiki.ros.org/xacro">
+  <xacro:include filename="$(find rto_description)/urdf/rto_parts.urdf.xacro"/>
+  <xacro:include filename="$(find rto_description)/urdf/rto_body.urdf.xacro"/>
   <xacro:include filename="$(find rto_description)/urdf/sensors/asus_xtion_pro.urdf.xacro"/>
   <xacro:include filename="$(find rto_description)/urdf/sensors/hokuyo.urdf.xacro"/>
-  <xacro:robotino_body/>
+  <xacro:rto_body/>
   <xacro:plate parent="base_link" name="plate"/>
   <xacro:bracket parent="base_link" name="bracket_hokuyo" scale="0.001">

File: rto_description/urdf/rto.urdf (robot description, URDF)
Before this commit: robot robotino, 7 links, 6 joints
Links:
- removed link platform_link
- link base_link: geometry collision cylinder length=0.05 radius=0.18; visual mesh filename=package://rto_description/meshes/parts/rto_base.dae scale=0.01 0.01 0.01
- link wheel0_link: geometry visual mesh filename=package://rto_description/meshes/parts/rto_wheel.dae scale=0.01 0.01 0.01
- link wheel1_link: geometry visual mesh filename=package://rto_description/meshes/parts/rto_wheel.dae scale=0.01 0.01 0.01
- link wheel2_link: geometry visual mesh filename=package://rto_description/meshes/parts/rto_wheel.dae scale=0.01 0.01 0.01
Joints:
- removed joint platform_joint

File: rto_description/urdf/rto_body.urdf.xacro (robot description, xacro)
@@ -6,6 +6,6 @@
     <xacro:property name="BASE_HEIGHT" value="0.05"/>
     <xacro:property name="BASE_MASS" value="20"/>
-    <!-- robotino_body -->
-    <xacro:macro name="robotino_body">
+    <!-- rto_body -->
+    <xacro:macro name="rto_body">
         <!-- base_link -->
         <link name="base_link">
@@ -20,5 +20,5 @@
                 <origin xyz="0.01 0 0" rpy="0 0 ${M_PI/2}"/>
                 <geometry>
-                    <mesh filename="package://rto_description/meshes/parts/robotino_base.dae"
+                    <mesh filename="package://rto_description/meshes/parts/rto_base.dae"
                         scale="${M_SCALE} ${M_SCALE} ${M_SCALE}"/>
                 </geometry>

File: rto_description/urdf/rto_parts.urdf.xacro (robot description, xacro)
@@ -19,5 +19,5 @@
                 <origin xyz="0 0 0" rpy="0 0 0"/>
                 <geometry>
-                    <mesh filename="package://rto_description/meshes/parts/robotino_wheel.dae" scale="${M_SCALE} ${M_SCALE} ${M_SCALE}"/>
+                    <mesh filename="package://rto_description/meshes/parts/rto_wheel.dae" scale="${M_SCALE} ${M_SCALE} ${M_SCALE}"/>
                 </geometry>
             </visual>

File: rto_description/urdf/rto_platform.urdf (robot description, URDF)
Before this commit: robot robotino, 6 links, 5 joints
Links:
- added link platform_link, mass 0.00001; visual cylinder length=0.02 radius=0.22; visual cylinder length=0.58 radius=0.04
- link base_link: geometry collision cylinder length=0.05 radius=0.18; visual mesh filename=package://rto_description/meshes/parts/rto_base.dae scale=0.01 0.01 0.01
- link wheel0_link: geometry visual mesh filename=package://rto_description/meshes/parts/rto_wheel.dae scale=0.01 0.01 0.01
- link wheel1_link: geometry visual mesh filename=package://rto_description/meshes/parts/rto_wheel.dae scale=0.01 0.01 0.01
- link wheel2_link: geometry visual mesh filename=package://rto_description/meshes/parts/rto_wheel.dae scale=0.01 0.01 0.01
Joints:
- added joint platform_joint: type fixed, parent base_link, child platform_link, origin xyz=0.0 0.0 0.13 rpy=0 0 0

File: rto_description/urdf/rto_platform_kinect.urdf (robot description, URDF)
Before this commit: robot robotino, 8 links, 7 joints
Links:
- link base_link: geometry collision cylinder length=0.05 radius=0.18; visual mesh filename=package://rto_description/meshes/parts/rto_base.dae scale=0.01 0.01 0.01
- link wheel0_link: geometry visual mesh filename=package://rto_description/meshes/parts/rto_wheel.dae scale=0.01 0.01 0.01
- link wheel1_link: geometry visual mesh filename=package://rto_description/meshes/parts/rto_wheel.dae scale=0.01 0.01 0.01
- link wheel2_link: geometry visual mesh filename=package://rto_description/meshes/parts/rto_wheel.dae scale=0.01 0.01 0.01

File: rto_description/urdf/rto_platform_kinect.urdf.xacro (robot description, xacro)
@@ -1,9 +1,9 @@
 <?xml version="1.0"?>
-<robot name="robotino" xmlns:xacro="http://wiki.ros.org/xacro">
-    <xacro:include filename="$(find rto_description)/urdf/robotino_body.urdf.xacro"/>
-    <xacro:include filename="$(find rto_description)/urdf/robotino_parts.urdf.xacro"/>
+<robot name="rto" xmlns:xacro="http://wiki.ros.org/xacro">
+    <xacro:include filename="$(find rto_description)/urdf/rto_body.urdf.xacro"/>
+    <xacro:include filename="$(find rto_description)/urdf/rto_parts.urdf.xacro"/>
     <xacro:include filename="$(find rto_description)/urdf/sensors/kinect.urdf.xacro"/>
-    <!-- main robotino body -->
-    <robotino_body/>
+    <!-- main rto body -->
+    <rto_body/>
     <!-- add platform -->
     <platform name="platform" parent="base_link">
