Commit message: Added new robots and updated rto-description structure

File: rto_description/urdf/robots/rto-2.urdf.xacro (robot description, xacro)
@@ -1,7 +1,7 @@
 <?xml version="1.0"?>
 <robot name="rto" xmlns:xacro="http://wiki.ros.org/xacro">
-  <xacro:include filename="$(find rto_description)/urdf/rto_parts.urdf.xacro"/>
-  <xacro:include filename="$(find rto_description)/urdf/rto_body.urdf.xacro"/>
-  <xacro:include filename="$(find rto_description)/urdf/sensors/asus_xtion_pro.urdf.xacro"/>
+  <xacro:include filename="$(find rto_description)/urdf/components/rto_parts.urdf.xacro"/>
+  <xacro:include filename="$(find rto_description)/urdf/components/rto_body.urdf.xacro"/>
+  <xacro:include filename="$(find rto_description)/urdf/sensors/realsense_d415.urdf.xacro"/>
   <xacro:include filename="$(find rto_description)/urdf/sensors/hokuyo.urdf.xacro"/>
   <xacro:rto_body/>
@@ -10,8 +10,7 @@
     <origin xyz="0.101 0 0.15" rpy="0 0 1.57"/>
   </xacro:bracket>
-  <xacro:bracket parent="base_link" name="bracket_camera" scale="0.000666666667">
-    <origin xyz="0.084 0 0.271" rpy="0 3.14 1.57"/>
-  </xacro:bracket>
-  <xacro:sensor_asus_xtion_pro parent="base_link"/>
+  <xacro:sensor_d415 name="d415" parent="base_link" use_nominal_extrinsics="true">
+    <origin xyz="0.061 0.0 0.271" rpy="0 0 0"/>
+  </xacro:sensor_d415>
   <xacro:hokuyo name="hokuyo" parent="base_link">
     <origin xyz="0.08 0 0.2015" rpy="0 0 0"/>
